File: PCB/swimate.sch (EAGLE design)
At the start: 18 parts, among them U1 USD-SOCKETNEW, U3 MCP73831

Commit message: Added SWD interface
Parts:
- added R3, R4: 24k, SparkFun-Passives:RESISTOR1206
- added R5, R6: (no value), SparkFun-Passives:RESISTOR1206
Connections:
- new net PIO_0: JTAG1.10
- new net PIO_10: JTAG1.4, R4.2
- new net PIO_15: JTAG1.2, R3.1
- new net PIO_9: JTAG1.6
- net 3.3V: now also JTAG1.1, R3.2, R5.2, R6.2
- net GND: now also JTAG1.3, JTAG1.5, JTAG1.7, JTAG1.9, R4.1
- net I2C_SCL: now also R6.1
- net I2C_SDA: now also R5.1
Other:
- moved on the sheet: C1, C2, C3, J1, JTAG1, LED1, R1, R2, U$1, U3

Commit message: Charge pump added
Parts:
- removed U4: (no value), microbuilder:LPC11U24_QFP64
- added C10, C8, C9: 0.1uF, SparkFun-Capacitors:CAP1206
- added C11, C12: 1uF, SparkFun-Capacitors:CAP1206
- added C13: .22uF, SparkFun-Capacitors:CAP1206
- added IC1: LPC11U24, mbed-HDK:LPC11U24
- added SJ1, SJ2: SOLDERJUMPERNO, SparkFun-Passives:SOLDERJUMPERNO
- added U5: DS3231MZ/V+T, maximparts:DS3231MZ/V+T
- added U6: MAX1595EUA33+, maximparts:MAX1595EUA33+
- added U7: MAX1811ESA-T, maximparts:MAX1811ESA-T
- added U8: MAX16054AZT+T, maximparts:MAX16054AZT+T
- added U9: HC_05, Bluetooth HC-05:HC_05
Connections:
- net SPI_MISO renamed SPI0_MISO
- net SPI_MOSI renamed SPI0_MOSI
- net SPI_SCK renamed SPI0_SCK
- new net 3V3_ENABLE: U6.*SHDN
- new net BT_KEY: SJ1.2, SJ2.2
- new net MCU_RX: IC1.PIO0.18/RXD/CT32B0M0, U9.TX
- new net MCU_TX: IC1.PIO0.19/TXD/CT32B0M1, U9.RX
- new net N$10: U9.RST
- new net N$11: SJ1.1, U9.PIO11
- new net N$12: C12.1, U6.AOUT, U6.OUT
- new net N$13: C13.1, U6.CXP
- new net N$14: C13.2, U6.CXN
- new net N$9: SJ2.1, U9.PIO3
- new net RST: U5.*RST
- new net VBAT: C2.2, C9.1, J1.+, U$1.IN, U3.VBAT, U5.VBAT
- net 3.3V: now also C10.1, C8.1, U5.VCC, U9.3V3
- net GND: now also C10.2, C11.2, C12.2, C8.2, C9.2, U5.GND, U6.GND, U6.PGND, U9.GND
- net I2C_SCL: now also U5.SCL
- net I2C_SDA: now also U5.SDA
- net N$1: now also C11.1, U6.IN; no longer C2.2, J1.+, U$1.IN, U3.VBAT
Other:
- note added: "Bluetooth Radio"
- note added: "Charge pump to 3v3"
- note added: "Micro SD"
- note added: "RTC"

Commit message: More improvements
Added bluetooth disable circuit and various other parts.
Parts:
- removed C3: 10uF, SparkFun-Capacitors:CAP1206
- removed J1: (no value), SparkFun-Connectors:JST_2MM_MALE
- removed JP1: USB-MICROB, SparkFun-Connectors:USB-MICROB
- removed LED1: (no value), SparkFun-LED:LED1206
- removed R1: 2k, SparkFun-Passives:RESISTOR1206
- removed R2: 470, SparkFun-Passives:RESISTOR1206
- removed U$1: V_REG_MIC2920, SparkFun-PowerIC:V_REG_MIC2920
- removed U3: MCP73831, SparkFun-PowerIC:MCP73831
- added C14: 4u7, SparkFun-Passives:CAP1206
- added C15: 0.1uF, SparkFun-Capacitors:CAP1206
- added C16, C17: 18pF, SparkFun-Capacitors:CAP1206
- added J2: (no value), SparkFun-Connectors:JST_2MM_MALE
- added JP2: (no value), SparkFun-Connectors:M08
- added JP3: USB-MICROB, SparkFun-Connectors:USB-MICROB
- added LED2: (no value), SparkFun-LED:LED1206
- added R10: 1k5, SparkFun-Passives:RESISTOR1206
- added R11, R12: 33, SparkFun-Passives:RESISTOR1206
- added R7: 470, SparkFun-Passives:RESISTOR1206
- added R8, R9: 10k, SparkFun-Passives:RESISTOR1206
- added SJ3: SOLDERJUMPERNO, SparkFun-Passives:SOLDERJUMPERNO
- added SW_PWR: (no value), SparkFun-Electromechanical:TAC_SWITCHKSA_SEALED
- added T1, T2: BSS84, mbed-HDK:BSS84
- added Y1: 12.000MHz, SparkFun-FreqCtrl:CRYSTAL5X3
- C1, C2: value 4u7 -> 18pF; device SparkFun-Passives:CAP1206 -> SparkFun-Capacitors:CAP1206
Connections:
- removed net N$2: R1.2, U3.PROG
- removed net N$3: LED1.C, R2.2
- removed net USB_DM: JP1.D-
- removed net USB_DP: JP1.D+
- new net BT_ENABLE: SJ3.2, T2.G
- new net CHARGE_STAT: LED2.C, U7.*CHG
- new net MPU_AD0: JP2.7, U2.AD0
- new net MPU_XCL: JP2.6, U2.E_SCL
- new net MPU_XDA: JP2.5, U2.E_SDA
- new net N$15: C8.1, R9.1, T2.S, U9.3V3
- new net N$16: R10.2, T1.D
- new net N$17: C17.1, IC1.USB_D+, R10.1, R12.1
- new net N$18: C16.1, IC1.USB_D-, R11.1
- new net N$19: JP3.D+, R12.2
- new net N$20: JP3.D-, R11.2
- new net N$21: IC1.PIO1.22/RI/MOSI1
- new net N$22: IC1.PIO1.20/DSR/SCK1
- new net N$23: C1.1, IC1.XTALIN, Y1.2
- new net N$24: C2.1, IC1.XTALOUT, Y1.1
- new net N$8: LED2.A, R7.1
- new net SYS_SHUTDOWN: R8.1, U8.CLEAR
- new net USB_SCON: T1.G
- net 3.3V: now also JP2.1, SJ3.1, T1.S, T2.D; no longer C3.1, C8.1, U$1.OUT, U9.3V3
- net 3V3_ENABLE: now also U8.OUT
- net GND: now also C14.1, C15.2, C16.2, C17.2, C2.2, J2.-, JP2.2, JP3.GND, R8.2, R9.2, SW_PWR.2, U7.GND, U7.GND_2, U7.SELI, U8.GND; no longer C2.1, C3.2, J1.-, JP1.GND, R1.1, R2.1, U$1.GND, U3.VSS
- net I2C_SCL: now also JP2.3
- net I2C_SDA: now also JP2.4
- net MPU_INT: now also JP2.8
- net N$1: now also SW_PWR.4, U8.IN; no longer C11.1, U6.IN
- net N$6: now also IC1.PIO1.21/DCD/MISO1; no longer LED1.A, U3.STAT
- net VBAT: now also C11.1, C14.2, J2.+, U6.IN, U7.BATT; no longer C2.2, J1.+, U$1.IN, U3.VBAT
- net VUSB: now also C15.1, JP3.VBUS, R7.2, U7.EN, U7.IN, U7.SELV, U8.VCC; no longer C1.1, JP1.VBUS, U3.VIN
Other:
- note added: "Li-Ion Charger"
- note added: "MPU-6050 Breakout connector"
- note added: "Realtime Clock"
- note removed: "RTC"
- moved on the sheet: C1, C2, U1, U7, U8

Commit message: Added dispaly
Parts:
- added C18, C19, C20, C3: (no value), SparkFun-Capacitors:CAP0805
- added C21: 2.2uF, SparkFun-Capacitors:CAP0805
- added C22: 10uF, SparkFun-Capacitors:CAP0805
- added R1: 390K, SparkFun-Passives:RESISTOR0805-RES
- added U$1: UG-2864HSWEG01, adafruit:UG-2864HSWEG01
Connections:
- new net N$2: C18.1, U$1.C1N
- new net N$25: C3.2, U$1.C2P
- new net N$26: C22.2, U$1.VCC
- new net N$27: C3.1, U$1.C2N
- new net N$28: C21.2, U$1.VCOMH
- new net N$29: C18.2, U$1.C1P
- new net N$3: R1.2, U$1.IREF
- new net SPI1_CS: U$1./CS
- new net SPI1_MOSI: U$1.D1/SCLK
- new net SPI1_SCK: U$1.D0/DI
- net 3.3V: now also C20.2, U$1.VDD
- net GND: now also C19.1, C20.1, C21.1, C22.1, R1.1, U$1.BS0, U$1.BS1, U$1.BS2, U$1.MT, U$1.MT2, U$1.VLSS, U$1.VSS
- net RST: now also U$1./RES
- net VBAT: now also C19.2, U$1.VBAT

Commit message: Starting Board layout.. still some pins to route
Parts:
- added C23, C24: 10uF, SparkFun-Capacitors:CAP1206
- added C25, C26: 100nF, SparkFun-Capacitors:CAP1206
- added R2: 2k, SparkFun-Passives:RESISTOR0805-RES
- added SJ4: (no value), SparkFun-Passives:SOLDERJUMPER_2WAYS
- added SJ5: SOLDERJUMPERNO, SparkFun-Passives:SOLDERJUMPERNO
- added SW_MODE: (no value), SparkFun-Electromechanical:TAC_SWITCHKSA_SEALED
- C10, C13, C15, C16, C17, C4, C5, C6, C7, C8, C9: device SparkFun-Capacitors:CAP1206 -> SparkFun-Passives:CAP0805
- JTAG1: device microbuilder:JTAG-CORTEXM3MOLEX -> microbuilder:JTAG-CORTEXM3
- R10, R11, R12, R3, R4: device SparkFun-Passives:RESISTOR1206 -> SparkFun-Passives:RESISTOR0805-RES
- R5, R6: value (none) -> 10k; device SparkFun-Passives:RESISTOR1206 -> SparkFun-Passives:RESISTOR0805-RES
- R8: value 10k -> 24k
- R9: value 10k -> 24K; device SparkFun-Passives:RESISTOR1206 -> SparkFun-Passives:RESISTOR0805-RES
Connections:
- net N$6 renamed SPI1_MISO
- removed net N$22: IC1.PIO1.20/DSR/SCK1
- removed net PIO_0: JTAG1.10
- removed net PIO_10: JTAG1.4, R4.2
- removed net PIO_15: JTAG1.2, R3.1
- removed net PIO_9: JTAG1.6
- new net BOOTLOAD: IC1.PIO0.1/CLKOUT/CT32B0M2/USB_FTOG, SJ5.2
- new net N$6: C23.1, C24.1, C25.1, C26.1, IC1.VDD@10, IC1.VDD@33, IC1.VDD@48, IC1.VDD@58
- new net SPI_MISO0: IC1.PIO0.8/MISO0/CT16B0M0
- new net SPI_MOSI0: IC1.PIO0.9/MOSI0/CT16B0M1, JTAG1.6
- new net SWCLK: IC1.SWCLK/PIO0.10/SCK0/CT16B0M2, JTAG1.4, R4.2
- new net SWDIO: IC1.SWDIO/PIO0.15/AD4/CT32B1M2, JTAG1.2, R3.1
- new net SW_MODE: SW_MODE.3, SW_MODE.4
- new net VDISPLAY: C19.2, SJ4.2, U$1.VBAT
- net 3.3V: now also SJ4.1
- net BT_ENABLE: no longer SJ3.2
- net GND: now also C16.1, C17.1, C23.2, C24.2, C25.2, C26.2, IC1.VSS@54, IC1.VSS@7, R2.1, SW_MODE.1, SW_MODE.2, SW_PWR.1; no longer C16.2, C17.2
- net I2C_SCL: now also IC1.PIO0.4/SCL(OD)
- net I2C_SDA: now also IC1.PIO0.5/SDA(OD)
- net N$1: now also SW_PWR.3
- net N$15: now also SJ3.2
- net N$17: now also C17.2; no longer C17.1
- net N$18: now also C16.2; no longer C16.1
- net N$21: now also R2.2, SJ5.1; no longer IC1.PIO1.22/RI/MOSI1
- net RST: now also IC1.PIO0.0/NRESET, JTAG1.10
- net SPI1_MOSI: now also IC1.PIO1.22/RI/MOSI1
- net SPI1_SCK: now also IC1.PIO1.20/DSR/SCK1
- net USB_SCON: now also IC1.PIO0.6/USB_CON/SCK0
- net VBAT: now also SJ4.3; no longer C19.2, U$1.VBAT
- net VUSB: now also IC1.PIO0.3/USB_VBUS
Other:
- moved on the sheet: C10, C11, C12, C13, C14, C15, C16, C17, C18, C19, C20, C21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

Commit message: More work on layout
Parts:
- C1, C2: device SparkFun-Capacitors:CAP1206 -> SparkFun-Passives:CAP0805
- C23, C24, C25, C26: device SparkFun-Capacitors:CAP1206 -> SparkFun-Capacitors:CAP0805
- R7, R8: device SparkFun-Passives:RESISTOR1206 -> SparkFun-Passives:RESISTOR0805-RES
Connections:
- removed net N$10: U9.RST
- net RST: now also U9.RST
Changed lines of the file:
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@@
 <grid distance="0.1" unitdist="inch" unit="inch" style="lines" multiple="1" display="no" altdistance="0.01" altunitdist="inch" altunit="inch"/>
 <layers>
-<layer number="1" name="Top" color="4" fill="1" visible="no" active="no"/>
-<layer number="16" name="Bottom" color="1" fill="1" visible="no" active="no"/>
-<layer number="17" name="Pads" color="2" fill="1" visible="no" active="no"/>
-<layer number="18" name="Vias" color="2" fill="1" visible="no" active="no"/>
-<layer number="19" name="Unrouted" color="6" fill="1" visible="no" active="no"/>
-<layer number="20" name="Dimension" color="15" fill="1" visible="no" active="no"/>
-<layer number="21" name="tPlace" color="7" fill="1" visible="no" active="no"/>
-<layer number="22" name="bPlace" color="7" fill="1" visible="no" active="no"/>
-<layer number="23" name="tOrigins" color="15" fill="1" visible="no" active="no"/>
-<layer number="24" name="bOrigins" color="15" fill="1" visible="no" active="no"/>
-<layer number="25" name="tNames" color="7" fill="1" visible="no" active="no"/>
-<layer number="26" name="bNames" color="7" fill="1" visible="no" active="no"/>
-<layer number="27" name="tValues" color="7" fill="1" visible="no" active="no"/>
-<layer number="28" name="bValues" color="7" fill="1" visible="no" active="no"/>
+<layer number="1" name="Top" color="4" fill="1" visible="yes" active="no"/>
+<layer number="16" name="Bottom" color="1" fill="1" visible="yes" active="no"/>
+<layer number="17" name="Pads" color="2" fill="1" visible="yes" active="no"/>
+<layer number="18" name="Vias" color="2" fill="1" visible="yes" active="no"/>
+<layer number="19" name="Unrouted" color="6" fill="1" visible="yes" active="no"/>
+<layer number="20" name="Dimension" color="15" fill="1" visible="yes" active="no"/>
+<layer number="21" name="tPlace" color="7" fill="1" visible="yes" active="no"/>
+<layer number="22" name="bPlace" color="7" fill="1" visible="yes" active="no"/>
+<layer number="23" name="tOrigins" color="15" fill="1" visible="yes" active="no"/>
+<layer number="24" name="bOrigins" color="15" fill="1" visible="yes" active="no"/>
+<layer number="25" name="tNames" color="7" fill="1" visible="yes" active="no"/>
+<layer number="26" name="bNames" color="7" fill="1" visible="yes" active="no"/>
+<layer number="27" name="tValues" color="7" fill="1" visible="yes" active="no"/>
+<layer number="28" name="bValues" color="7" fill="1" visible="yes" active="no"/>
 <layer number="29" name="tStop" color="7" fill="3" visible="no" active="no"/>
 <layer number="30" name="bStop" color="7" fill="6" visible="no" active="no"/>
@@
 <layer number="35" name="tGlue" color="7" fill="4" visible="no" active="no"/>
 <layer number="36" name="bGlue" color="7" fill="5" visible="no" active="no"/>
-<layer number="37" name="tTest" color="7" fill="1" visible="no" active="no"/>
-<layer number="38" name="bTest" color="7" fill="1" visible="no" active="no"/>
+<layer number="37" name="tTest" color="7" fill="1" visible="yes" active="no"/>
+<layer number="38" name="bTest" color="7" fill="1" visible="yes" active="no"/>
 <layer number="39" name="tKeepout" color="4" fill="11" visible="no" active="no"/>
 <layer number="40" name="bKeepout" color="1" fill="11" visible="no" active="no"/>
@@
 <layer number="44" name="Drills" color="7" fill="1" visible="no" active="no"/>
 <layer number="45" name="Holes" color="7" fill="1" visible="no" active="no"/>
-<layer number="46" name="Milling" color="3" fill="1" visible="no" active="no"/>
-<layer number="47" name="Measures" color="7" fill="1" visible="no" active="no"/>
-<layer number="48" name="Document" color="7" fill="1" visible="no" active="no"/>
-<layer number="49" name="Reference" color="7" fill="1" visible="no" active="no"/>
-<layer number="50" name="dxf" color="7" fill="1" visible="no" active="no"/>
-<layer number="51" name="tDocu" color="7" fill="1" visible="no" active="no"/>
-<layer number="52" name="bDocu" color="7" fill="1" visible="no" active="no"/>
-<layer number="53" name="tGND_GNDA" color="7" fill="9" visible="no" active="no"/>
-<layer number="54" name="bGND_GNDA" color="1" fill="9" visible="no" active="no"/>
-<layer number="56" name="wert" color="7" fill="1" visible="no" active="no"/>
-<layer number="57" name="tCAD" color="7" fill="1" visible="no" active="no"/>
+<layer number="46" name="Milling" color="3" fill="1" visible="yes" active="no"/>
+<layer number="47" name="Measures" color="7" fill="1" visible="yes" active="no"/>
+<layer number="48" name="Document" color="7" fill="1" visible="yes" active="no"/>
+<layer number="49" name="Reference" color="7" fill="1" visible="yes" active="no"/>
+<layer number="50" name="dxf" color="7" fill="1" visible="yes" active="no"/>
+<layer number="51" name="tDocu" color="7" fill="1" visible="yes" active="no"/>
+<layer number="52" name="bDocu" color="7" fill="1" visible="yes" active="no"/>
+<layer number="53" name="tGND_GNDA" color="7" fill="9" visible="yes" active="no"/>
+<layer number="54" name="bGND_GNDA" color="1" fill="9" visible="yes" active="no"/>
+<layer number="56" name="wert" color="7" fill="1" visible="yes" active="no"/>
+<layer number="57" name="tCAD" color="7" fill="1" visible="yes" active="no"/>
 <layer number="91" name="Nets" color="2" fill="1" visible="yes" active="yes"/>
 <layer number="92" name="Busses" color="1" fill="1" visible="yes" active="yes"/>
@@
 <part name="GND23" library="SparkFun-Aesthetics" deviceset="GND" device=""/>
 <part name="LED2" library="SparkFun-LED" deviceset="LED" device="1206"/>
-<part name="R7" library="SparkFun-Passives" deviceset="RESISTOR" device="1206" value="470"/>
+<part name="R7" library="SparkFun-Passives" deviceset="RESISTOR" device="0805-RES" value="470"/>
 <part name="GND24" library="SparkFun-Aesthetics" deviceset="GND" device=""/>
 <part name="C15" library="SparkFun-Passives" deviceset="CAP" device="0805" value="0.1uF"/>
 <part name="GND25" library="SparkFun-Aesthetics" deviceset="GND" device=""/>
 <part name="SW_PWR" library="SparkFun-Electromechanical" deviceset="TAC_SWITCH" device="KSA_SEALED"/>
-<part name="R8" library="SparkFun-Passives" deviceset="RESISTOR" device="1206" value="24k"/>
+<part name="R8" library="SparkFun-Passives" deviceset="RESISTOR" device="0805-RES" value="24k"/>
 <part name="GND26" library="SparkFun-Aesthetics" deviceset="GND" device=""/>
 <part name="T1" library="mbed-HDK" deviceset="BSS84" device=""/>
@@
 <part name="C17" library="SparkFun-Passives" deviceset="CAP" device="0805" value="18pF"/>
 <part name="Y1" library="SparkFun-FreqCtrl" deviceset="CRYSTAL" device="5X3" value="12.000MHz"/>
-<part name="C1" library="SparkFun-Capacitors" deviceset="CAP" device="1206" value="18pF"/>
-<part name="C2" library="SparkFun-Capacitors" deviceset="CAP" device="1206" value="18pF"/>
+<part name="C1" library="SparkFun-Passives" deviceset="CAP" device="0805" value="18pF"/>
+<part name="C2" library="SparkFun-Passives" deviceset="CAP" device="0805" value="18pF"/>
 <part name="GND1" library="SparkFun-Aesthetics" deviceset="GND" device=""/>
 <part name="GND2" library="SparkFun-Aesthetics" deviceset="GND" device=""/>
@@
 <part name="GND30" library="SparkFun-Aesthetics" deviceset="GND" device=""/>
 <part name="SUPPLY1" library="SparkFun-Aesthetics" deviceset="3.3V" device=""/>
-<part name="C23" library="SparkFun-Capacitors" deviceset="CAP" device="1206" value="10uF"/>
-<part name="C24" library="SparkFun-Capacitors" deviceset="CAP" device="1206" value="10uF"/>
-<part name="C25" library="SparkFun-Capacitors" deviceset="CAP" device="1206" value="100nF"/>
-<part name="C26" library="SparkFun-Capacitors" deviceset="CAP" device="1206" value="100nF"/>
+<part name="C23" library="SparkFun-Capacitors" deviceset="CAP" device="0805" value="10uF"/>
+<part name="C24" library="SparkFun-Capacitors" deviceset="CAP" device="0805" value="10uF"/>
+<part name="C25" library="SparkFun-Capacitors" deviceset="CAP" device="0805" value="100nF"/>
+<part name="C26" library="SparkFun-Capacitors" deviceset="CAP" device="0805" value="100nF"/>
 <part name="GND11" library="SparkFun-Aesthetics" deviceset="GND" device=""/>
 <part name="SJ4" library="SparkFun-Passives" deviceset="SOLDERJUMPER_2WAY" device="S"/>
@@
 <label x="-132.08" y="99.06" size="1.778" layer="95"/>
 </segment>
-</net>
-<net name="N$10" class="0">
 <segment>
 <pinref part="U9" gate="G$1" pin="RST"/>
 <wire x1="-20.32" y1="-60.96" x2="-25.4" y2="-60.96" width="0.1524" layer="91"/>
-</segment>
-</net>
+<label x="-25.4" y="-60.96" size="1.778" layer="95"/>
+</segment>
+</net>
