File: PCB/swimate_display.brd (EAGLE design)
At the start: 69.5 x 34.3 mm, 53 parts, among them IC1 LPC11U24, T1 BSS84, T2 BSS84, U1 USD-SOCKETNEW, U5 DS3231MZ/V+T, U6 MAX1595EUA33+, U7 MAX1811ESA-T, U8 MAX16054AZT+T, U9 HC_05, Y1 12.000MHz

Commit message: changed pcb size and separated display portion
Parts:
- added R1: 10k, SparkFun-Passives:0603-RES
- added R13: 24k, SparkFun-Passives:0603-RES
- moved C1 31.3 mm to (24.1, 25.1)
- moved Y1 23.9 mm to (30.2, 17.3), turned to 90 degrees
- moved SW_MODE 22.4 mm to (6.60, 5.84)
- moved R4 21.8 mm to (54.4, 32.3), turned to 90 degrees
- moved R8 17.0 mm to (23.4, 7.62), turned to 180 degrees
- moved JTAG1 12.3 mm to (61.7, 28.7), flipped to the bottom
- moved C2 12.2 mm to (30.7, 8.89), turned to 270 degrees
- moved SW_PWR 11.7 mm to (23.4, 11.4), turned to 270 degrees
- moved U8 11.7 mm to (23.4, 11.4), turned to 90 degrees
- moved C15 11.6 mm to (25.9, 12.7), turned to 180 degrees
- moved R3 9.52 mm to (51.8, 31.2)
- moved C5 6.12 mm to (17.0, 3.56)
- moved C6 5.59 mm to (13.5, 4.06)
- moved R5 5.29 mm to (23.6, 4.57)
- moved C4 3.66 mm to (21.1, 3.05)
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Connections:
- new net VBATTMON: R1.1, R13.2
- net GND: now also R13.1
- net VBAT: now also R1.2
Routing:
- net GND: track 89.9 -> 208.8 mm, vias 2 -> 8
- net RST: track 0.00 -> 44.6 mm, vias 0 -> 1
- net N$6: track 0.00 -> 42.4 mm, vias 0 -> 1
- net N$24: track 0.00 -> 28.0 mm, vias 0 -> 2
- net VBAT: track 2.88 -> 26.7 mm
- net I2C_SDA: track 39.8 -> 20.6 mm
- net MCU_TX: track 0.00 -> 16.4 mm
- net N$23: track 3.69 -> 19.4 mm
- net BOOTLOAD: track 0.00 -> 12.3 mm
- net N$12: track 0.00 -> 11.5 mm
- net MCU_RX: track 0.00 -> 9.83 mm
- net 3V3_ENABLE: track 18.7 -> 26.8 mm
- net N$15: track 20.5 -> 27.2 mm
- net 3.3V: track 26.8 -> 31.1 mm
- net N$14: track 0.00 -> 3.97 mm
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