File: PCB/swimate_displayext.brd (EAGLE design)
At the start: 50.9 x 51.2 mm, 56 parts, among them IC1 LPC11U24, J1 FTSH-105-01-L-DV, T1 BSS84, T2 BSS84, U1 USD-SOCKETNEW, U3 NC7SV86P5X, U5 DS3231MZ/V+T, U6 MAX1595EUA33+, U7 MAX1811ESA-T, U8 MAX16054AZT+T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

Commit message: display board update
Connections:
- net GND: no longer J1.6
- net SPI0_MISO: now also J1.6
Changed lines of the file:
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@@
 <wire x1="26.416" y1="39.751" x2="26.416" y2="40.329078125" width="0.4064" layer="1"/>
 <wire x1="26.416" y1="40.329078125" x2="26.277096875" y2="40.46798125" width="0.4064" layer="1"/>
-<contactref element="J1" pad="6"/>
 <contactref element="J1" pad="8"/>
 <contactref element="J1" pad="10"/>
@@
 <wire x1="-4.318" y1="6.985" x2="1.132" y2="5.588" width="0" layer="19" extent="1-16"/>
 <wire x1="-5.588" y1="6.985" x2="-4.318" y2="6.985" width="0" layer="19" extent="1-1"/>
-<wire x1="-6.858" y1="6.985" x2="-5.588" y2="6.985" width="0" layer="19" extent="1-1"/>
 </signal>
 <signal name="3.3V">
@@
 <wire x1="32.512" y1="21.082" x2="33.604" y2="21.082" width="0.254" layer="1"/>
 <wire x1="33.604" y1="21.082" x2="33.64" y2="21.118" width="0.254" layer="1"/>
+<contactref element="J1" pad="6"/>
+<wire x1="-6.858" y1="6.985" x2="10.89" y2="36.63" width="0" layer="19" extent="1-16"/>
 </signal>
 <signal name="SD_DETECT">
