File: PCB/swimate_displayext.sch (EAGLE design)
At the start: 55 parts, among them IC1 LPC11U24, T1 BSS84, T2 BSS84, U1 USD-SOCKETNEW, U5 DS3231MZ/V+T, U6 MAX1595EUA33+, U7 MAX1811ESA-T, U8 MAX16054AZT+T, U9 HC_05, Y1 12.000MHz

Commit message: Passed DRC
TODO: DRC, connect CS signals for display and SD card.
TODO: replace connector for display board.
Connections:
- removed net SCK0: IC1.SWCLK/PIO0.10/SCK0/CT16B0M2, JTAG1.4, R4.2
- net BT_ENABLE: now also IC1.PIO1.13/DTR/CT16B0M1/TXD
- net BT_KEY: now also IC1.TDO/PIO0.13/AD2/CB32B1M0
- net GND: now also J2.PAD1, J2.PAD2
- net SPI0_SCK: now also IC1.SWCLK/PIO0.10/SCK0/CT16B0M2, JTAG1.4, R4.2
- net SW_MODE: now also IC1.PIO1.17/CT16B0C1/RXD, SW_MODE.3; no longer SW_MODE.4
Changed lines of the file:
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@@
 <part name="SUPPLY12" library="SparkFun-Aesthetics" deviceset="3.3V" device=""/>
 <part name="SUPPLY9" library="SparkFun-Aesthetics" deviceset="3.3V" device=""/>
+<part name="GND30" library="SparkFun-Aesthetics" deviceset="GND" device=""/>
 </parts>
 <sheets>
@@
 <instance part="SUPPLY12" gate="G$1" x="-101.6" y="55.88"/>
 <instance part="SUPPLY9" gate="G$1" x="-58.42" y="114.3"/>
+<instance part="GND30" gate="1" x="-256.54" y="12.7"/>
 </instances>
 <busses>
@@
 <pinref part="JP2" gate="G$1" pin="1"/>
 <wire x1="203.2" y1="30.48" x2="198.12" y2="30.48" width="0.1524" layer="91"/>
+<label x="195.58" y="30.48" size="1.778" layer="95"/>
 </segment>
 </net>
@@
 <pinref part="GND26" gate="1" pin="GND"/>
 <wire x1="-274.32" y1="71.12" x2="-274.32" y2="68.58" width="0.1524" layer="91"/>
+</segment>
+<segment>
+<pinref part="J2" gate="G$1" pin="PAD1"/>
+<wire x1="-246.38" y1="17.78" x2="-251.46" y2="17.78" width="0.1524" layer="91"/>
+<wire x1="-251.46" y1="17.78" x2="-251.46" y2="25.4" width="0.1524" layer="91"/>
+<wire x1="-251.46" y1="25.4" x2="-236.22" y2="25.4" width="0.1524" layer="91"/>
+<wire x1="-236.22" y1="25.4" x2="-236.22" y2="17.78" width="0.1524" layer="91"/>
+<pinref part="J2" gate="G$1" pin="PAD2"/>
+<wire x1="-236.22" y1="17.78" x2="-238.76" y2="17.78" width="0.1524" layer="91"/>
+<pinref part="GND30" gate="1" pin="GND"/>
+<wire x1="-251.46" y1="17.78" x2="-256.54" y2="17.78" width="0.1524" layer="91"/>
+<wire x1="-256.54" y1="17.78" x2="-256.54" y2="15.24" width="0.1524" layer="91"/>
+<junction x="-251.46" y="17.78"/>
 </segment>
 </net>
@@
 <label x="-162.56" y="-48.26" size="1.778" layer="95"/>
 </segment>
+<segment>
+<pinref part="IC1" gate="G$1" pin="SWCLK/PIO0.10/SCK0/CT16B0M2"/>
+<wire x1="-38.1" y1="43.18" x2="-45.72" y2="43.18" width="0.1524" layer="91"/>
+<label x="-50.8" y="43.18" size="1.778" layer="95"/>
+</segment>
+<segment>
+<pinref part="JTAG1" gate="G$1" pin="4"/>
+<wire x1="-139.7" y1="106.68" x2="-134.62" y2="106.68" width="0.1524" layer="91"/>
+<pinref part="R4" gate="G$1" pin="2"/>
+<wire x1="-134.62" y1="106.68" x2="-129.54" y2="106.68" width="0.1524" layer="91"/>
+<wire x1="-134.62" y1="106.68" x2="-134.62" y2="96.52" width="0.1524" layer="91"/>
+<junction x="-134.62" y="106.68"/>
+<label x="-132.08" y="106.68" size="1.778" layer="95"/>
+</segment>
 </net>
 <net name="SPI0_MISO" class="0">
@@
 <wire x1="48.26" y1="-55.88" x2="43.18" y2="-55.88" width="0.1524" layer="91"/>
 <label x="48.26" y="-45.72" size="1.778" layer="95"/>
+</segment>
+<segment>
+<pinref part="IC1" gate="G$1" pin="TDO/PIO0.13/AD2/CB32B1M0"/>
+<wire x1="-38.1" y1="35.56" x2="-50.8" y2="35.56" width="0.1524" layer="91"/>
+<label x="-50.8" y="35.56" size="1.778" layer="95"/>
 </segment>
 </net>
@@
 <wire x1="-50.8" y1="-58.42" x2="-38.1" y2="-58.42" width="0.1524" layer="91"/>
 </segment>
+<segment>
+<pinref part="IC1" gate="G$1" pin="PIO1.13/DTR/CT16B0M1/TXD"/>
+<wire x1="55.88" y1="81.28" x2="68.58" y2="81.28" width="0.1524" layer="91"/>
+<label x="58.42" y="81.28" size="1.778" layer="95"/>
+</segment>
 </net>
 <net name="N$16" class="0">
@@
 </segment>
 </net>
-<net name="SCK0" class="0">
-<segment>
-<pinref part="IC1" gate="G$1" pin="SWCLK/PIO0.10/SCK0/CT16B0M2"/>
-<wire x1="-38.1" y1="43.18" x2="-45.72" y2="43.18" width="0.1524" layer="91"/>
-<label x="-50.8" y="43.18" size="1.778" layer="95"/>
-</segment>
-<segment>
-<pinref part="JTAG1" gate="G$1" pin="4"/>
-<wire x1="-139.7" y1="106.68" x2="-134.62" y2="106.68" width="0.1524" layer="91"/>
-<pinref part="R4" gate="G$1" pin="2"/>
-<wire x1="-134.62" y1="106.68" x2="-129.54" y2="106.68" width="0.1524" layer="91"/>
-<wire x1="-134.62" y1="106.68" x2="-134.62" y2="96.52" width="0.1524" layer="91"/>
-<junction x="-134.62" y="106.68"/>
-<label x="-132.08" y="106.68" size="1.778" layer="95"/>
-</segment>
-</net>
 <net name="BOOTLOAD" class="0">
 <segment>
@@
 <net name="SW_MODE" class="0">
 <segment>
-<pinref part="SW_MODE" gate="S" pin="4"/>
-<wire x1="-243.84" y1="-38.1" x2="-231.14" y2="-38.1" width="0.1524" layer="91"/>
 <label x="-238.76" y="-38.1" size="1.778" layer="95"/>
+<pinref part="SW_MODE" gate="S" pin="3"/>
+<wire x1="-238.76" y1="-38.1" x2="-231.14" y2="-38.1" width="0.1524" layer="91"/>
+<wire x1="-243.84" y1="-35.56" x2="-238.76" y2="-35.56" width="0.1524" layer="91"/>
+<wire x1="-238.76" y1="-35.56" x2="-238.76" y2="-38.1" width="0.1524" layer="91"/>
+</segment>
+<segment>
+<pinref part="IC1" gate="G$1" pin="PIO1.17/CT16B0C1/RXD"/>
+<wire x1="55.88" y1="63.5" x2="66.04" y2="63.5" width="0.1524" layer="91"/>
+<label x="58.42" y="63.5" size="1.778" layer="95"/>
 </segment>
 </net>
@@
 </sheet>
 </sheets>
+<errors>
+</errors>
 </schematic>
 </drawing>

Commit message: Added CS pins and turn off logic (MCU safe powerdown for SD card
Parts:
- added U3: NC7SV86P5X, Fairchild_By_element14_Batch_1:NC7SV86P5X
Connections:
- new net N$2: U3.A, U8.OUT
- new net PO_DISABLE: IC1.TDO/PIO0.13/AD2/CB32B1M0, U3.B
- net 3V3_ENABLE: now also U3.Y; no longer U8.OUT
- net BT_KEY: now also IC1.NTRST/PIO0.14/AD3/CT32B1M1; no longer IC1.TDO/PIO0.13/AD2/CB32B1M0
- net DISP_CS: now also IC1.PIO1.25/CT32B0M1
- net DISP_DC: now also IC1.PIO1.0/CT32B1M0
- net GND: now also U3.GND
- net SD_CS: now also IC1.PIO1.19/DTR/SSEL1
- net VBAT: now also U3.VCC
Other:
- moved on the sheet: C15, SJ4, SW_PWR, U8
Changed lines of the file:
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@@
 <?xml version="1.0" encoding="utf-8"?>
 <!DOCTYPE eagle SYSTEM "eagle.dtd">
-<eagle version="6.5.0">
+<eagle version="6.4">
 <drawing>
 <settings>
@@
 <part name="SUPPLY9" library="SparkFun-Aesthetics" deviceset="3.3V" device=""/>
 <part name="GND30" library="SparkFun-Aesthetics" deviceset="GND" device=""/>
+<part name="U3" library="Fairchild_By_element14_Batch_1" deviceset="NC7SV86P5X" device=""/>
+<part name="GND33" library="SparkFun-Aesthetics" deviceset="GND" device=""/>
 </parts>
 <sheets>
@@
 <instance part="U6" gate="A" x="-185.42" y="50.8"/>
 <instance part="U7" gate="A" x="-292.1" y="48.26"/>
-<instance part="U8" gate="A" x="-266.7" y="86.36"/>
+<instance part="U8" gate="A" x="-320.04" y="119.38"/>
 <instance part="U9" gate="G$1" x="2.54" y="-50.8"/>
 <instance part="IC1" gate="G$1" x="-2.54" y="63.5"/>
@@
 <instance part="LED2" gate="G$1" x="-228.6" y="55.88"/>
 <instance part="R7" gate="G$1" x="-233.68" y="63.5" rot="R180"/>
-<instance part="GND24" gate="1" x="-297.18" y="76.2"/>
-<instance part="C15" gate="G$1" x="-182.88" y="81.28"/>
-<instance part="GND25" gate="1" x="-182.88" y="73.66"/>
-<instance part="SW_PWR" gate="S" x="-289.56" y="93.98"/>
-<instance part="GND26" gate="1" x="-274.32" y="66.04"/>
+<instance part="GND24" gate="1" x="-350.52" y="109.22"/>
+<instance part="C15" gate="G$1" x="-236.22" y="114.3"/>
+<instance part="GND25" gate="1" x="-236.22" y="106.68"/>
+<instance part="SW_PWR" gate="S" x="-342.9" y="127"/>
+<instance part="GND26" gate="1" x="-327.66" y="93.98"/>
 <instance part="T1" gate="G$1" x="73.66" y="-5.08"/>
 <instance part="T2" gate="G$1" x="-33.02" y="-55.88"/>
@@
 <instance part="SUPPLY11" gate="G$1" x="114.3" y="81.28" rot="R180"/>
 <instance part="GND29" gate="1" x="187.96" y="71.12"/>
-<instance part="SJ4" gate="1" x="-274.32" y="76.2" rot="R90"/>
+<instance part="SJ4" gate="1" x="-327.66" y="109.22" rot="R90"/>
 <instance part="SUPPLY12" gate="G$1" x="-101.6" y="55.88"/>
 <instance part="SUPPLY9" gate="G$1" x="-58.42" y="114.3"/>
 <instance part="GND30" gate="1" x="-256.54" y="12.7"/>
+<instance part="U3" gate="A" x="-213.36" y="83.82"/>
+<instance part="GND33" gate="1" x="-236.22" y="71.12"/>
 </instances>
 <busses>
@@
 <segment>
 <pinref part="U8" gate="A" pin="VCC"/>
-<label x="-203.2" y="86.36" size="1.778" layer="95"/>
+<label x="-256.54" y="119.38" size="1.778" layer="95"/>
 <pinref part="C15" gate="G$1" pin="1"/>
-<wire x1="-205.74" y1="86.36" x2="-182.88" y2="86.36" width="0.1524" layer="91"/>
+<wire x1="-259.08" y1="119.38" x2="-236.22" y2="119.38" width="0.1524" layer="91"/>
 </segment>
 <segment>
@@
 <wire x1="203.2" y1="30.48" x2="198.12" y2="30.48" width="0.1524" layer="91"/>
 <label x="195.58" y="30.48" size="1.778" layer="95"/>
+</segment>
+<segment>
+<pinref part="U3" gate="A" pin="VCC"/>
+<wire x1="-231.14" y1="86.36" x2="-238.76" y2="86.36" width="0.1524" layer="91"/>
+<label x="-238.76" y="86.36" size="1.778" layer="95"/>
 </segment>
 </net>
@@
 <pinref part="U8" gate="A" pin="GND"/>
 <pinref part="GND24" gate="1" pin="GND"/>
-<wire x1="-266.7" y1="83.82" x2="-297.18" y2="83.82" width="0.1524" layer="91"/>
-<wire x1="-297.18" y1="83.82" x2="-297.18" y2="78.74" width="0.1524" layer="91"/>
+<wire x1="-320.04" y1="116.84" x2="-350.52" y2="116.84" width="0.1524" layer="91"/>
+<wire x1="-350.52" y1="116.84" x2="-350.52" y2="111.76" width="0.1524" layer="91"/>
 <pinref part="SW_PWR" gate="S" pin="2"/>
-<wire x1="-294.64" y1="91.44" x2="-297.18" y2="91.44" width="0.1524" layer="91"/>
-<wire x1="-297.18" y1="91.44" x2="-297.18" y2="83.82" width="0.1524" layer="91"/>
-<junction x="-297.18" y="83.82"/>
+<wire x1="-347.98" y1="124.46" x2="-350.52" y2="124.46" width="0.1524" layer="91"/>
+<wire x1="-350.52" y1="124.46" x2="-350.52" y2="116.84" width="0.1524" layer="91"/>
+<junction x="-350.52" y="116.84"/>
 </segment>
 <segment>
 <pinref part="C15" gate="G$1" pin="2"/>
 <pinref part="GND25" gate="1" pin="GND"/>
-<wire x1="-182.88" y1="78.74" x2="-182.88" y2="76.2" width="0.1524" layer="91"/>
+<wire x1="-236.22" y1="111.76" x2="-236.22" y2="109.22" width="0.1524" layer="91"/>
 </segment>
 <segment>
@@
 <pinref part="SJ4" gate="1" pin="1"/>
 <pinref part="GND26" gate="1" pin="GND"/>
-<wire x1="-274.32" y1="71.12" x2="-274.32" y2="68.58" width="0.1524" layer="91"/>
+<wire x1="-327.66" y1="104.14" x2="-327.66" y2="96.52" width="0.1524" layer="91"/>
 </segment>
 <segment>
@@
 <wire x1="-256.54" y1="17.78" x2="-256.54" y2="15.24" width="0.1524" layer="91"/>
 <junction x="-251.46" y="17.78"/>
+</segment>
+<segment>
+<pinref part="GND33" gate="1" pin="GND"/>
+<pinref part="U3" gate="A" pin="GND"/>
+<wire x1="-236.22" y1="73.66" x2="-231.14" y2="73.66" width="0.1524" layer="91"/>
 </segment>
 </net>
@@
 <label x="93.98" y="-40.64" size="1.778" layer="95"/>
 </segment>
+<segment>
+<pinref part="IC1" gate="G$1" pin="PIO1.19/DTR/SSEL1"/>
+<wire x1="55.88" y1="58.42" x2="66.04" y2="58.42" width="0.1524" layer="91"/>
+<label x="60.96" y="58.42" size="1.778" layer="95"/>
+</segment>
 </net>
 <net name="SPI0_MOSI" class="0">
@@
 </segment>
 <segment>
-<pinref part="IC1" gate="G$1" pin="TDO/PIO0.13/AD2/CB32B1M0"/>
-<wire x1="-38.1" y1="35.56" x2="-50.8" y2="35.56" width="0.1524" layer="91"/>
-<label x="-50.8" y="35.56" size="1.778" layer="95"/>
+<pinref part="IC1" gate="G$1" pin="NTRST/PIO0.14/AD3/CT32B1M1"/>
+<wire x1="-38.1" y1="33.02" x2="-50.8" y2="33.02" width="0.1524" layer="91"/>
+<label x="-53.34" y="33.02" size="1.778" layer="95"/>
 </segment>
 </net>
@@
 <wire x1="-185.42" y1="48.26" x2="-198.12" y2="48.26" width="0.1524" layer="91"/>
 <label x="-203.2" y="48.26" size="1.778" layer="95"/>
-<wire x1="-198.12" y1="48.26" x2="-198.12" y2="83.82" width="0.1524" layer="91"/>
-<pinref part="U8" gate="A" pin="OUT"/>
-<wire x1="-198.12" y1="83.82" x2="-205.74" y2="83.82" width="0.1524" layer="91"/>
-<label x="-203.2" y="83.82" size="1.778" layer="95"/>
+<pinref part="U3" gate="A" pin="Y"/>
+<wire x1="-195.58" y1="86.36" x2="-190.5" y2="86.36" width="0.1524" layer="91"/>
+<wire x1="-190.5" y1="86.36" x2="-190.5" y2="71.12" width="0.1524" layer="91"/>
+<wire x1="-190.5" y1="71.12" x2="-198.12" y2="71.12" width="0.1524" layer="91"/>
+<wire x1="-198.12" y1="71.12" x2="-198.12" y2="48.26" width="0.1524" layer="91"/>
+<junction x="-198.12" y="48.26"/>
 </segment>
 </net>
@@
 <segment>
 <pinref part="U8" gate="A" pin="CLEAR"/>
-<wire x1="-266.7" y1="81.28" x2="-274.32" y2="81.28" width="0.1524" layer="91"/>
-<label x="-287.02" y="81.28" size="1.778" layer="95"/>
+<wire x1="-320.04" y1="114.3" x2="-327.66" y2="114.3" width="0.1524" layer="91"/>
+<label x="-340.36" y="114.3" size="1.778" layer="95"/>
 <pinref part="SJ4" gate="1" pin="2"/>
 </segment>
@@
 <segment>
 <pinref part="SW_PWR" gate="S" pin="4"/>
-<wire x1="-284.48" y1="91.44" x2="-274.32" y2="91.44" width="0.1524" layer="91"/>
-<wire x1="-274.32" y1="91.44" x2="-274.32" y2="86.36" width="0.1524" layer="91"/>
+<wire x1="-337.82" y1="124.46" x2="-327.66" y2="124.46" width="0.1524" layer="91"/>
+<wire x1="-327.66" y1="124.46" x2="-327.66" y2="119.38" width="0.1524" layer="91"/>
 <pinref part="U8" gate="A" pin="IN"/>
-<wire x1="-274.32" y1="86.36" x2="-266.7" y2="86.36" width="0.1524" layer="91"/>
+<wire x1="-327.66" y1="119.38" x2="-320.04" y2="119.38" width="0.1524" layer="91"/>
 </segment>
 </net>
@@
 <segment>
 <pinref part="IC1" gate="G$1" pin="PIO1.13/DTR/CT16B0M1/TXD"/>
-<wire x1="55.88" y1="81.28" x2="68.58" y2="81.28" width="0.1524" layer="91"/>
+<wire x1="55.88" y1="81.28" x2="66.04" y2="81.28" width="0.1524" layer="91"/>
 <label x="58.42" y="81.28" size="1.778" layer="95"/>
 </segment>
@@
 <label x="-160.02" y="-50.8" size="1.778" layer="95"/>
 </segment>
+<segment>
+<pinref part="IC1" gate="G$1" pin="PIO1.25/CT32B0M1"/>
+<wire x1="55.88" y1="40.64" x2="66.04" y2="40.64" width="0.1524" layer="91"/>
+<label x="60.96" y="40.64" size="1.778" layer="95"/>
+</segment>
 </net>
 <net name="DISP_DC" class="0">
@@
 <wire x1="-144.78" y1="-55.88" x2="-160.02" y2="-55.88" width="0.1524" layer="91"/>
 <label x="-160.02" y="-55.88" size="1.778" layer="95"/>
+</segment>
+<segment>
+<pinref part="IC1" gate="G$1" pin="PIO1.0/CT32B1M0"/>
+<wire x1="55.88" y1="114.3" x2="68.58" y2="114.3" width="0.1524" layer="91"/>
+<label x="58.42" y="114.3" size="1.778" layer="95"/>
 </segment>
 </net>
@@
 </segment>
 </net>
+<net name="N$2" class="0">
+<segment>
+<pinref part="U8" gate="A" pin="OUT"/>
+<label x="-256.54" y="116.84" size="1.778" layer="95"/>
+<wire x1="-259.08" y1="116.84" x2="-241.3" y2="116.84" width="0.1524" layer="91"/>
+<wire x1="-241.3" y1="116.84" x2="-241.3" y2="81.28" width="0.1524" layer="91"/>
+<pinref part="U3" gate="A" pin="A"/>
+<wire x1="-241.3" y1="81.28" x2="-231.14" y2="81.28" width="0.1524" layer="91"/>
+</segment>
+</net>
+<net name="PO_DISABLE" class="0">
+<segment>
+<pinref part="IC1" gate="G$1" pin="TDO/PIO0.13/AD2/CB32B1M0"/>
+<wire x1="-38.1" y1="35.56" x2="-50.8" y2="35.56" width="0.1524" layer="91"/>
+<label x="-53.34" y="35.56" size="1.778" layer="95"/>
+</segment>
+<segment>
+<pinref part="U3" gate="A" pin="B"/>
+<wire x1="-231.14" y1="78.74" x2="-248.92" y2="78.74" width="0.1524" layer="91"/>
+<label x="-246.38" y="78.74" size="1.778" layer="95"/>
+</segment>
+</net>
